File: remote/hardware/ib4/ib4.kicad_pcb (KiCad board)
At the start: 4 copper layers, 24 parts, among them J1 Conn_01x02_Female, J10 Screw_Terminal_01x03, J2 Screw_Terminal_01x02, J3 Conn_01x01_Female, J4 Conn_01x01_Female, J5 Conn_01x01_Female, J6 Screw_Terminal_01x03, J7 Screw_Terminal_01x03, J8 Screw_Terminal_01x03, J9 Screw_Terminal_01x03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

Commit message: update
Parts:
- moved R2 33.3 mm to (121.1, 65.7)
- moved J7 32.4 mm to (95.3, 59.6)
- moved J6 31.5 mm to (95.6, 75.7)
- moved J8 31.1 mm to (95.4, 44.3)
- moved Q1 28.1 mm to (109.5, 81.8)
- moved R1 27.5 mm to (115.8, 79.2), turned to 270 degrees
- moved Q2 26.9 mm to (128.9, 68.5), turned to 270 degrees
- moved R3 20.0 mm to (109.6, 71.2)
- moved J5 12.6 mm to (121.8, 80.8), turned to 270 degrees
- moved J4 11.3 mm to (121.8, 85.4), turned to 180 degrees
- moved J3 10.6 mm to (128.8, 80.8), turned to 180 degrees
- moved U1 4.05 mm to (119.5, 29.3)
Routing:
- net GND: track 359.0 -> 273.7 mm, vias 0 -> 4
- net +3V3: track 189.9 -> 254.8 mm, vias 4 -> 2
- net RX: track 17.7 -> 56.9 mm
- net D12: track 62.1 -> 94.0 mm, vias 4 -> 2
- net 5V_BOOST: track 92.3 -> 79.5 mm, vias 0 -> 2
- net DECAGON_SWITCH: track 53.5 -> 62.3 mm
- net Net-(Q1-Pad3): track 7.95 -> 13.7 mm
- net 5V_SWITCHED: track 14.1 -> 9.19 mm
- net A0: track 18.9 -> 22.5 mm
- net Net-(Q1-Pad2): track 9.47 -> 6.32 mm
- net LI-ION: track 23.3 -> 24.3 mm
- net A1: track 19.3 -> 20.0 mm
- net TIMER: track 30.3 -> 29.6 mm

Commit message: update
Parts:
- moved H3 236.2 mm to (8.00, 6.00)
- moved H2 232.4 mm to (8.00, 72.0)
- moved H4 165.7 mm to (90.0, 6.00)
- moved H1 144.0 mm to (90.0, 72.0)
- moved J1 85.8 mm to (51.6, 27.0)
- moved J10 85.8 mm to (88.2, 50.3)
- moved J8 85.8 mm to (13.2, 19.4)
- moved J9 85.8 mm to (88.2, 64.8)
- moved JP2 85.8 mm to (56.5, 36.0)
- moved JP4 85.8 mm to (71.7, 36.0)
- moved Q1 85.8 mm to (27.4, 57.0)
- moved R1 85.8 mm to (33.6, 54.2)
- moved U1 85.8 mm to (37.4, 4.40)
- moved U3 85.8 mm to (80.5, 10.6)
- moved J2 85.8 mm to (26.9, 5.00)
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Routing:
- net GND: track 273.7 -> 273.1 mm
Other:
- board outline added: 97 x 76.8 mm

Commit message: update
Other:
- board size 97 x 76.8 mm -> 97 x 77 mm
Changed lines of the file:
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@@
   (general
     (thickness 1.6)
-    (drawings 9)
+    (drawings 8)
     (tracks 252)
     (zones 0)
@@
     (visible_elements FFFFFF7F)
     (pcbplotparams
-      (layerselection 0x00000_fffffff8)
+      (layerselection 0x01000_fffffff8)
       (usegerberextensions false)
       (usegerberattributes false)
@@
       (viasonmask false)
       (mode 1)
-      (useauxorigin false)
+      (useauxorigin true)
       (hpglpennumber 1)
       (hpglpenspeed 20)
       (hpglpendiameter 15.000000)
-      (psnegative true)
+      (psnegative false)
       (psa4output false)
       (plotreference false)
@@
       (padsonsilk false)
       (subtractmaskfromsilk false)
-      (outputformat 5)
+      (outputformat 1)
       (mirror false)
-      (drillshape 1)
+      (drillshape 0)
       (scaleselection 1)
-      (outputdirectory "svg/"))
+      (outputdirectory "mill_v"))
   )
   (net 0 "")
@@
     )
   )
-  (gr_line (start 0 0) (end 96.95 0) (layer Edge.Cuts) (width 0.05))
+  (gr_line (start 0 0) (end 96 0) (layer Edge.Cuts) (width 0.05))
   (gr_line (start 96.95 1.6) (end 96.95 0) (layer Edge.Cuts) (width 0.05))
-  (gr_line (start 0 76.75) (end 1.1 76.75) (layer Edge.Cuts) (width 0.05))
-  (gr_line (start 0 0) (end 0 76.75) (layer Edge.Cuts) (width 0.05))
+  (gr_line (start 0 0) (end 0 77) (layer Edge.Cuts) (width 0.05))
   (gr_line (start 31.65 18.95) (end 32.4 18.95) (layer Edge.Cuts) (width 0.05))
-  (gr_line (start 96.95 76.75) (end 1.1 76.75) (layer Edge.Cuts) (width 0.05))
-  (gr_line (start 96.95 1.6) (end 96.95 76.75) (layer Edge.Cuts) (width 0.05))
+  (gr_line (start 96 77) (end 0 77) (layer Edge.Cuts) (width 0.05))
+  (gr_line (start 96 0) (end 96 77) (layer Edge.Cuts) (width 0.05))
   (dimension 4.55 (width 0.1) (layer Dwgs.User)
     (gr_text "4.550 mm" (at 29.35 58.225 90) (layer Dwgs.User)

Commit message: update
Other:
- board size 97 x 77 mm -> 96 x 77 mm
Changed lines of the file:
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@@
   (general
     (thickness 1.6)
-    (drawings 8)
+    (drawings 6)
     (tracks 252)
     (zones 0)
@@
   )
   (gr_line (start 0 0) (end 96 0) (layer Edge.Cuts) (width 0.05))
-  (gr_line (start 96.95 1.6) (end 96.95 0) (layer Edge.Cuts) (width 0.05))
   (gr_line (start 0 0) (end 0 77) (layer Edge.Cuts) (width 0.05))
-  (gr_line (start 31.65 18.95) (end 32.4 18.95) (layer Edge.Cuts) (width 0.05))
   (gr_line (start 96 77) (end 0 77) (layer Edge.Cuts) (width 0.05))
   (gr_line (start 96 0) (end 96 77) (layer Edge.Cuts) (width 0.05))
