File: gateway/hardware/ib4/ib4.kicad_pcb (KiCad board)
At the start: 4 copper layers, 96 x 77 mm, 14 parts, among them J1 Conn_01x02_Female, J6 Screw_Terminal_01x03, J7 Screw_Terminal_01x03, J8 Screw_Terminal_01x03, U1 bme280, U2 tpl5110, U3 lora_breakout

Commit message: update
Parts:
- moved J1 8.46 mm to (52.5, 36.6)
- moved J6 8.46 mm to (18.7, 57.4)
- moved J8 8.46 mm to (18.5, 26.0)
- moved JP2 8.46 mm to (61.8, 42.6)
- moved JP4 8.46 mm to (77.0, 42.6)
- moved R3 8.46 mm to (32.7, 53.0)
- moved U1 8.46 mm to (34.5, 18.4)
- moved U2 8.46 mm to (32.2, 28.7)
- moved U3 8.46 mm to (85.8, 17.2)
- moved J7 8.46 mm to (18.4, 41.3)
