File: greenhouse/remote/v4/remote/remote.kicad_pcb (KiCad board)
At the start: 2 copper layers, 66 x 71.1 mm, 17 parts, among them J1 Conn_01x03_Female, J10 Conn_01x04_Female, J2 Screw_Terminal_01x03, J3 Conn_01x04_Female, J4 Screw_Terminal_01x04, J5 Conn_01x02_Female, J6 Conn_01x12_Male, J7 Conn_01x16_Female, J8 Screw_Terminal_01x02, J9 Adafruit BME280

Commit message: update
Parts:
- added G***: LOGO, remote:vlogS, F.Cu at (136.7, 107.4)
- moved J2 2.00 mm to (87.4, 85.9)
- moved J8 1.84 mm to (87.4, 103.6)
- moved J4 1.70 mm to (87.4, 58.8)
- moved R1 1.70 mm to (94.1, 79.7)
- moved J1 1.70 mm to (95.5, 88.5)
- moved J5 1.40 mm to (95.5, 105.4)
- moved J10 1.27 mm to (95.4, 70.8)
Routing:
- net +3V3: track 0.00 -> 180.2 mm, vias 0 -> 1
- net GND: track 0.00 -> 155.9 mm, vias 0 -> 2
- net SDA: track 0.00 -> 77.9 mm
- net SCL: track 0.00 -> 73.6 mm, vias 0 -> 2
- net Net-(J1-Pad2): track 0.00 -> 39.2 mm
- net Net-(J5-Pad2): track 0.00 -> 32.3 mm
Other:
- board text added: "3V"
- board text added: "D12"
- board text added: "GND"
- board text added: "SCL"
- board text added: "SDA"
- board text added: "VIN"
- board text added: "http://pvos.org/lama-remote"
- board text added: "v4"
