File: greenhouse/remote/v5/remote/remote.kicad_pcb (KiCad board)
At the start: 2 copper layers, 66 x 71.1 mm, 18 parts, among them J1 Conn_01x03_Female, J10 Conn_01x04_Female, J2 Screw_Terminal_01x03, J3 Conn_01x04_Female, J4 Screw_Terminal_01x04, J5 Conn_01x02_Female, J6 Conn_01x12_Male, J7 Conn_01x16_Female, J8 Screw_Terminal_01x02, J9 Adafruit BME280

Commit message: update
Parts:
- removed the G*** at (136.7, 107.4)
- added G***: LOGO, remote:pvos7, F.Cu at (135.9, 91.9)
Other:
- board text added: "http://pvos.org"
